Commit message: Update robot_core.xacro

File: src/capstone_description/urdf/robot_core.xacro (robot description, xacro)
@@ -20,7 +20,16 @@
     <link name="base_link">
     </link>
+    <!-- BASE FOOTPRINT -->
+    <link name="base_footprint">
+    </link>
+    <!-- Joint to connect base_link to base_footprint -->
+    <joint name="base_footprint_joint" type="fixed">
+        <parent link="base_link"/>
+        <child link="base_footprint"/>
+        <origin xyz="0 0 0" rpy="0 0 0"/>
+    </joint>
     <!-- CHASSIS LINK -->
     <joint name="chassis_joint" type="fixed">
-        <parent link="base_link"/>
+        <parent link="base_footprint"/>
         <child link="chassis"/>
         <origin xyz="-0.1 0 0"/>
@@ -44,7 +53,7 @@
         </xacro:inertial_box>
     </link>
-    <!-- LEFT WHEEK LINK -->
+    <!-- LEFT WHEEL LINK -->
     <joint name="left_wheel_joint" type="continuous">
-        <parent link="base_link"/>
+        <parent link="base_footprint"/>
         <child link="left_wheel"/>
         <origin xyz="0 0.175 0" rpy="-${pi/2} 0 0"/>
@@ -67,7 +76,7 @@
         </xacro:inertial_cylinder>
     </link>
-    <!-- RIGHT WHEEK LINK -->
+    <!-- RIGHT WHEEL LINK -->
     <joint name="right_wheel_joint" type="continuous">
-        <parent link="base_link"/>
+        <parent link="base_footprint"/>
         <child link="right_wheel"/>
         <origin xyz="0 -0.175 0" rpy="${pi/2} 0 0"/>
